File: tamagotchi/tamagotchi.kicad_pcb (KiCad board)
At the start: 2 copper layers, 7 parts, among them SW1 SW_Push, SW2 SW_Push, SW3 SW_Push, U1 XIAO-ESP32-C3-SMD, U2 HS96L03W2C03

Commit message: added blender
Parts:
- added G***: LOGO, JINX:JINX, F.Cu at (150.5, 97.0)
- added G***: LOGO, JINX:JINX, B.Cu at (149.0, 113.0)
- added REF**: MountingHole_3.2mm_M3, MountingHole:MountingHole_3.2mm_M3, F.Cu at (173.5, 110.3)
- added REF**: MountingHole_3.2mm_M3, MountingHole:MountingHole_3.2mm_M3, F.Cu at (126.5, 110.0)
- BUZZER1, U1: moved to B.Cu
- moved BT1 97.8 mm to (149.3, 69.8), turned to 90 degrees
- moved BUZZER1 60.7 mm to (153.4, 97.7), turned to 180 degrees
- moved U2 44.5 mm to (150.0, 87.4)
- moved SW3 44.5 mm to (167.5, 122.5)
- moved SW1 38.6 mm to (133.3, 122.5)
- moved SW2 35.9 mm to (150.8, 124.0)
- moved U1 26.9 mm to (150.8, 128.0), turned to -90 degrees
Connections:
- SW2 pad 2: Net-(U1-GPIO2_A0_D0) -> Net-(U1-GPIO3_A1_D1)
- U1 pad 2: Net-(U1-GPIO2_A0_D0) -> Net-(U1-GPIO3_A1_D1)
Routing:
- net +BATT: track 0.00 -> 61.1 mm
- net +3V3: track 0.00 -> 46.4 mm
- net Net-(U1-GPIO7_D5_SCL): track 0.00 -> 41.1 mm
- net Net-(U1-GPIO21_D6_TX): track 0.00 -> 40.7 mm
- net Net-(U1-GPIO2_A0_D0): track 0.00 -> 38.2 mm
- net Net-(BUZZER1-+): track 0.00 -> 32.0 mm
- net Net-(U1-GPIO3_A1_D1): track 0.00 -> 16.2 mm
- net Net-(U1-GPIO4_A2_D2): track 0.00 -> 12.0 mm
- added copper zone on B.Cu, net GND
- added copper zone on F.Cu, net GND
Other:
- board outline added: 65 x 74.8 mm
