File: tamagotchi/tamagotchi.kicad_sch (KiCad schematic)
At the start: 7 parts, among them SW1 SW_Push, SW2 SW_Push, SW3 SW_Push, U1 XIAO-ESP32-C3-SMD, U2 HS96L03W2C03

Commit message: added blender
Connections:
- net at SW2.2, U1.2 (GPIO3_A1_D1): no longer SW3.2, U1.1 (GPIO2_A0_D0)
- new net: SW3.2, U1.1 (GPIO2_A0_D0)
- no-connect marks 0 -> 11
Changed lines of the file:
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@@
 	(paper "A4")
-	(junction
-		(at 88.9 99.06)
-		(diameter 0)
-		(color 0 0 0 0)
-	)
-	(junction
-		(at 88.9 102.87)
-		(diameter 0)
-		(color 0 0 0 0)
-	)
 	(junction
 		(at 78.74 111.76)
@@
 		(color 0 0 0 0)
 	)
+	(no_connect
+		(at 146.05 80.01)
+	)
+	(no_connect
+		(at 138.43 80.01)
+	)
+	(no_connect
+		(at 134.62 80.01)
+	)
+	(no_connect
+		(at 161.29 118.11)
+	)
+	(no_connect
+		(at 119.38 114.3)
+	)
+	(no_connect
+		(at 161.29 114.3)
+	)
+	(no_connect
+		(at 142.24 80.01)
+	)
+	(no_connect
+		(at 149.86 80.01)
+	)
+	(no_connect
+		(at 119.38 110.49)
+	)
+	(no_connect
+		(at 130.81 80.01)
+	)
+	(no_connect
+		(at 161.29 121.92)
+	)
 	(wire
 		(pts
@@
 	(wire
 		(pts
-			(xy 88.9 109.22) (xy 119.38 109.22)
+			(xy 88.9 109.22) (xy 111.76 109.22)
 		)
 		(stroke
@@
 	(wire
 		(pts
-			(xy 119.38 109.22) (xy 119.38 106.68)
+			(xy 111.76 106.68) (xy 119.38 106.68)
+		)
+		(stroke
+			(width 0)
+			(type default)
+		)
+	)
+	(wire
+		(pts
+			(xy 111.76 109.22) (xy 111.76 106.68)
 		)
 		(stroke
@@
 	(wire
 		(pts
-			(xy 114.3 115.57) (xy 114.3 116.84)
-		)
-		(stroke
-			(width 0)
-			(type default)
-		)
-	)
-	(wire
-		(pts
 			(xy 132.08 147.32) (xy 132.08 151.13)
 		)
@@
 		(pts
 			(xy 161.29 102.87) (xy 170.18 102.87)
-		)
-		(stroke
-			(width 0)
-			(type default)
-		)
-	)
-	(wire
-		(pts
-			(xy 88.9 99.06) (xy 88.9 102.87)
 		)
 		(stroke
@@
 		(in_pos_files yes)
 		(dnp no)
-		(fields_autoplaced yes)
 		(property "Reference" "U2"
 			(at 91.44 115.5699 0)
@@
 		)
 		(property "Value" "HS96L03W2C03"
-			(at 91.44 118.1099 0)
+			(at 102.87 124.968 0)
 			(show_name no)
 			(do_not_autoplace no)
@@
 	(symbol
 		(lib_id "power:+3V3")
-		(at 114.3 116.84 0)
+		(at 114.3 115.57 0)
 		(unit 1)
 		(body_style 1)
@@
 		(dnp no)
 		(property "Reference" "#PWR07"
-			(at 114.3 120.65 0)
+			(at 114.3 119.38 0)
 			(hide yes)
 			(show_name no)
@@
 		)
 		(property "Value" "+3V3"
-			(at 114.554 116.586 0)
+			(at 111.76 112.014 0)
 			(show_name no)
 			(do_not_autoplace no)
@@
 		)
 		(property "Footprint" ""
-			(at 114.3 116.84 0)
+			(at 114.3 115.57 0)
 			(hide yes)
 			(show_name no)
@@
 		)
 		(property "Datasheet" ""
-			(at 114.3 116.84 0)
+			(at 114.3 115.57 0)
 			(hide yes)
 			(show_name no)
@@
 		)
 		(property "Description" "Power symbol creates a global label with name \"+3V3\""
-			(at 114.3 116.84 0)
-			(hide yes)
-			(show_name no)
+			(at 114.3 115.57 0)
+			(hide yes)
+			(show_name no)
